Commit message: go2_description integrated to nav pkg.

File: go2_description/urdf/go2_description.urdf (robot description, URDF)
Before this commit: robot go2_description, 42 links, 41 joints
Links:
- removed link base
- added link base_link, mass 6.921; collision box size=0.3762 0.0935 0.114; visual mesh filename=package://go2_description/dae/base.dae
Joints:
- joint FL_hip_joint: parent base -> base_link
- joint FL_hip_rotor_joint: parent base -> base_link
- joint FR_hip_joint: parent base -> base_link
- joint FR_hip_rotor_joint: parent base -> base_link
- joint Head_upper_joint: parent base -> base_link
- joint RL_hip_joint: parent base -> base_link
- joint RL_hip_rotor_joint: parent base -> base_link
- joint RR_hip_joint: parent base -> base_link
- joint RR_hip_rotor_joint: parent base -> base_link
- joint front_camera_joint: parent base -> base_link
- joint imu_joint: parent base -> base_link
- joint radar_joint: parent base -> base_link

File: go2_description/xacro/robot.xacro (robot description, xacro)
@@ -17,8 +17,8 @@
             <origin rpy="0 0 0" xyz="0 0 0"/>
             <parent link="world"/>
-            <child link="base"/>
+            <child link="base_link"/>
         </joint>
     </xacro:if>
-    <link name="base">
+    <link name="base_link">
         <visual>
             <origin rpy="0 0 0" xyz="0 0 0"/>
@@ -30,5 +30,5 @@
     <joint name="floating_base" type="fixed">
         <origin rpy="0 0 0" xyz="0 0 0"/>
-        <parent link="base"/>
+        <parent link="base_link"/>
         <child link="trunk"/>
     </joint>
@@ -55,4 +55,11 @@
                 izz="${trunk_izz}"/>
         </inertial>
+    </link>
+    <joint name="lidar_joint" type="fixed">
+        <parent link="trunk"/>
+        <child link="utlidar_lidar"/>
+        <origin rpy="0 0 0" xyz="0.32715 -0.00003 -0.04297"/>
+    </joint>
+    <link name="utlidar_lidar">
     </link>
     <joint name="imu_joint" type="fixed">
