Commit message: Base-footprint.

File: go2_description/xacro/robot.xacro (robot description, xacro)
@@ -63,4 +63,12 @@
     <link name="utlidar_lidar">
     </link>
+    <!-- Todo: NEed to account for the calf joint angle and projected height of the calf.. -->
+    <joint name="base_footprint_joint" type="fixed">
+        <parent link="trunk"/>
+        <child link="base_footprint"/>
+        <origin rpy="0 0 0" xyz="0.0 0.0 -0.213"/>
+    </joint>
+    <link name="base_footprint">
+    </link>
     <joint name="imu_joint" type="fixed">
         <parent link="trunk"/>
